File: Physical/BoomerAmp/MB_boomer_amp.kicad_pcb (KiCad board)
At the start: 2 copper layers, 43.2 x 33 mm, 12 parts

Commit message: Add logo to the Boomer amp.  Part of #86
Parts:
- added G***: LOGO, mcqn-kicad-lib:miab-logo-9x7mm, F.Cu at (162.6, 117.5)
- added G***: LOGO, mcqn-kicad-lib:miab-logo-9x7mm, B.Cu at (162.6, 117.5)
Other:
- board text added: "museuminabox.org"
